File: kicad/OpenWatch.sch (KiCad schematic (older format))
At the start: 1 part

Commit message: Basic schematic layout
Parts:
- removed U?: STM32F303RCT6, Housings_QFP:LQFP-64_10x10mm_Pitch0.5mm, symbol STM32F303RCT6
- added C? (x11): 100nF, symbol C_Small
- added C? (x2): 1uF, symbol C_Small
- added C?: 10uF, symbol C_Small
- added C? (x2): 18pF, symbol C_Small
- added D? (x2): LED, symbol LED
- added FP?: BM71BLES1FC2, symbol BM71BLES1FC2
- added J?: USB_microB_2040002-1, symbol USB_microB_2040002-1
- added J?: JTAG, symbol Conn_02x05_Odd_Even
- added J?: Conn_01x05, symbol Conn_01x05
- added R? (x11): 10K, symbol R
- added R?: 4.75K, symbol R
- added R?: 402, symbol R
- added R? (x3): 100K, symbol R
- added R?: 1K, symbol R
- added U?: LSM6DSL, symbol LSM6DSL
- added U?: RT9818A-18GV, symbol RT9818A-18GV
- added U?: STM32F303RCT6, symbol STM32F303RCT6
- added U?: AT42QT1070-MMHR, symbol AT42QT1070-MMHR
- added U?: WM1389CT-ND, symbol WM1389CT-ND
- added Y?: Crystal_GND24, symbol Crystal_GND24
Connections:
- net labels added: +3.3V, +5V, DISP_SCLK, DISP_SCS, DISP_SDI, GND, IMU_SCL, IMU_SDI, IMU_SDO, KEY_0, KEY_1, KEY_2, KEY_3, KEY_4, NRST_TOUCH, RX_BLE, STM_NRST, TCK, TDO, TMS, TOUCH_0, TOUCH_1, TOUCH_2, TOUCH_3, TOUCH_4, TX_BLE
- wire segments 0 -> 192
- no-connect marks 0 -> 45
Other:
- note added: "-What is EXTCOMIN used for?\n-How do we verify the pitch for the FPC?\n"

Commit message: Adds power management IC configuration
Parts:
- removed J?: JTAG, symbol Conn_02x05_Odd_Even
- removed J?: Conn_01x05, symbol Conn_01x05
- added BT?: Battery, symbol Battery
- added C? (x2): 4.7uF, symbol C_Small
- added C?: 1uF, symbol C_Small
- added D? (x2): Led_Small, symbol Led_Small
- added P?: CONN_02X05, symbol CONN_02X05
- added P?: CONN_01X05, symbol CONN_01X05
- added R? (x2): 1.5K, symbol R_Small
- added R?: 56.2K, symbol R
- added R? (x2): R, symbol R
- added R?: 3.06K, symbol R
- added R?: 10K, symbol R
- added U?: bq24232rgtr, symbol bq24232rgtr
Connections:
- net labels added: +BATT, D+, D-, VBUS
- wire segments 192 -> 254
- no-connect marks 45 -> 46
Other:
- note added: "Input Current Limit = 500 mA\nCharge Failsafe Timer = 7.5 h\nCV Termination Current = Depends on battery\nFast Charge Current = Depends on battery"
- note added: "JTAG"
- note added: "LiPoly Coin Cell or Pouch Cell"

Commit message: Fixes schematic to 4.07 KICAD
Parts:
- removed D? (x2): Led_Small, symbol Led_Small
- removed P?: CONN_02X05, symbol CONN_02X05
- removed P?: CONN_01X05, symbol CONN_01X05
- added D? (x2): LED, symbol LED_Small
- added J?: Conn_01x05, symbol Conn_01x05
- added J?: Conn_02x05_Odd_Even, symbol Conn_02x05_Odd_Even

Commit message: Adds additional components to BOM
Parts:
- added R?: 10K, symbol R
- added SW?: SW_Push, symbol SW_Push
Connections:
- wire segments 254 -> 257
Changed lines of the file:
@@
 L GND #PWR?
 U 1 1 59FBDDD8
-P 2150 6950
-F 0 "#PWR?" H 2150 6700 50  0001 C CNN
-F 1 "GND" H 2150 6800 50  0000 C CNN
-F 2 "" H 2150 6950 50  0001 C CNN
-F 3 "" H 2150 6950 50  0001 C CNN
-	1    2150 6950
+P 2150 7300
+F 0 "#PWR?" H 2150 7050 50  0001 C CNN
+F 1 "GND" H 2150 7150 50  0000 C CNN
+F 2 "" H 2150 7300 50  0001 C CNN
+F 3 "" H 2150 7300 50  0001 C CNN
+	1    2150 7300
 	1    0    0    -1
 $EndComp
@@
 	2150 6950 2150 6850
 Wire Wire Line
-	2150 6850 2300 6850
+	1600 6850 2300 6850
 $Comp
 L Crystal_GND24 Y?
@@
 	1    0    0    -1
 $EndComp
+$Comp
+L R R?
+U 1 1 59FE11A8
+P 2150 7100
+F 0 "R?" V 2230 7100 50  0000 C CNN
+F 1 "10K" V 2150 7100 50  0000 C CNN
+F 2 "" V 2080 7100 50  0001 C CNN
+F 3 "" H 2150 7100 50  0001 C CNN
+	1    2150 7100
+	1    0    0    -1
+$EndComp
+Wire Wire Line
+	2150 7250 2150 7300
+$Comp
+L SW_Push SW?
+U 1 1 59FE1E31
+P 1400 6850
+F 0 "SW?" H 1450 6950 50  0000 L CNN
+F 1 "SW_Push" H 1400 6790 50  0000 C CNN
+F 2 "" H 1400 7050 50  0001 C CNN
+F 3 "" H 1400 7050 50  0001 C CNN
+	1    1400 6850
+	1    0    0    -1
+$EndComp
+Connection ~ 2150 6850
+$Comp
+L +3.3V #PWR?
+U 1 1 59FE205C
+P 1150 6750
+F 0 "#PWR?" H 1150 6600 50  0001 C CNN
+F 1 "+3.3V" H 1150 6890 50  0000 C CNN
+F 2 "" H 1150 6750 50  0001 C CNN
+F 3 "" H 1150 6750 50  0001 C CNN
+	1    1150 6750
+	1    0    0    -1
+$EndComp
+Wire Wire Line
+	1150 6750 1150 6850
+Wire Wire Line
+	1150 6850 1200 6850
 $EndSCHEMATC

Commit message: Finalizes certain schematic elements
Parts:
- removed BT?: Battery, symbol Battery
- removed C? (x2): 4.7uF, symbol C_Small
- removed C?: 1uF, symbol C_Small
- removed D? (x2): LED, symbol LED_Small
- removed R? (x2): 1.5K, symbol R_Small
- removed R?: 56.2K, symbol R
- removed R? (x2): R, symbol R
- removed R?: 3.06K, symbol R
- removed R?: 10K, symbol R
- removed U?: STM32F303RCT6, symbol STM32F303RCT6
- removed U?: bq24232rgtr, symbol bq24232rgtr
- added C? (x3): 1uF, symbol C_Small
- added C? (x2): C, symbol C
- added D?: BAT54, symbol D_Schottky
- added J?: Vibration Motor, symbol Conn_01x02
- added Q?: RUM002N02T2L, symbol Q_NMOS_GSD
- added SW?: SW_Push, symbol SW_Push
- added U?: STM32F303RCT6-48, symbol STM32F303RCT6-48
- added U?: TPS60241DGKR, symbol TPS60241DGKR
- added Y?: Crystal, symbol Crystal
Connections:
- net labels added: 5V_EN, MOTOR_EN
- net labels removed: VBUS
- wire segments 257 -> 254
- no-connect marks 46 -> 26
Other:
- note added: "BLE"
- note added: "Capacitive Touch\n"
- note added: "IMU\n"
- note added: "JTAG Breakout"
- note added: "OLED Display\n\n"
- note added: "TODO: Find a better charge pump\nwith lower power consumption\n\n"
- note added: "Vibration Motor\n"
- note removed: "Input Current Limit = 500 mA\nCharge Failsafe Timer = 7.5 h\nCV Termination Current = Depends on battery\nFast Charge Current = Depends on battery"
- note removed: "LiPoly Coin Cell or Pouch Cell"

Commit message: Finishes first implementation of the schematic
Parts:
- added BT?: Battery_Cell, symbol Battery_Cell
- added C?: 10uF, symbol C_Small
- added C?: 2.2uF, symbol C_Small
- added C?: 1uF, symbol C_Small
- added C? (x3): 4.7uF, symbol C_Small
- added D?: LED, symbol LED
- added J?: Conn_01x03, symbol Conn_01x03
- added J? (x2): Conn_01x02, symbol Conn_01x02
- added R?: 20K, symbol R
- added R? (x2): 10K, symbol R
- added R?: 402, symbol R
- added R?: 470, symbol R
- added U?: TPS2112APWR, symbol TPS2112APWR
- added U?: TSP70933DBVR, symbol TSP70933DBVR
- added U?: MCP73831T-2ACI, symbol MCP73831T-2ACI
Connections:
- net labels added: VBATT, VUSB
- net labels removed: +BATT
- wire segments 254 -> 311
Other:
- note added: "Battery\n"
- note added: "Bypass Capacitors\n"
- note added: "Charging\n"
- note added: "Microcontroller\n"
- note added: "Multiplex & Regulate\n"
- note added: "microUSB\n"

Commit message: Adds crystals and fixes minor schematic issues
Parts:
- added Q? (x2): RUM002N02T2L, symbol Q_NMOS_GSD
- C? (x2): value C -> 12.5pF
- R?: value 20K -> 200K
- R?: value 10K -> 100K
- Y?: value Crystal_GND24 -> FA-238
- Y?: value Crystal -> ECS.327
Connections:
- net labels added: BATT_EN
- wire segments 311 -> 319
- no-connect marks 26 -> 25
Other:
- note added: "Allow for\ncompletely\nturning off \nthe battery\n"

Commit message: Fixes some schematic issues and adds a 3-color LED
Parts:
- removed D?: LED, symbol LED
- added D2: LED_ARGB, symbol LED_ARGB
- added R7, R9: 1K, symbol R
- R25: renamed from R?; value 402 -> 1K
- gave numbers to parts that had none: 77
Connections:
- net labels added: IMU_CS, IMU_INT_1, IMU_INT_2, LED_BLUE, LED_GREEN, LED_RED
- wire segments 319 -> 331
- no-connect marks 25 -> 19
