File: kicad/OpenWatch.sch (KiCad schematic (older format))
At the start: 81 parts, among them J1 USB_microB_2040002-1, J2 Conn_01x02, J3 Conn_02x05_Odd_Even, J4 Vibration Motor, J5 Conn_01x03, J6 Conn_01x05, J7 Conn_01x02, Q1 RUM002N02T2L, Q2 RUM002N02T2L, Q3 RUM002N02T2L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

Commit message: Fixes pull-up issues with JTAG wiring
Parts:
- removed R11, R12, R13: 100K, symbol R
Connections:
- net labels added: TDI
- wire segments 331 -> 325
- no-connect marks 19 -> 17
Changed lines of the file:
@@
 L +3.3V #PWR013
 U 1 1 59FB260A
-P 9700 9650
-F 0 "#PWR013" H 9700 9500 50  0001 C CNN
-F 1 "+3.3V" H 9700 9790 50  0000 C CNN
-F 2 "" H 9700 9650 50  0001 C CNN
-F 3 "" H 9700 9650 50  0001 C CNN
-	1    9700 9650
-	1    0    0    -1
-$EndComp
-Wire Wire Line
-	9950 9800 9700 9800
-Wire Wire Line
-	9700 9800 9700 9650
+P 9700 9350
+F 0 "#PWR013" H 9700 9200 50  0001 C CNN
+F 1 "+3.3V" H 9700 9490 50  0000 C CNN
+F 2 "" H 9700 9350 50  0001 C CNN
+F 3 "" H 9700 9350 50  0001 C CNN
+	1    9700 9350
+	1    0    0    -1
+$EndComp
+Wire Wire Line
+	9950 9500 9700 9500
+Wire Wire Line
+	9700 9500 9700 9350
 $Comp
 L GND #PWR014
 U 1 1 59FB2824
-P 9400 10100
-F 0 "#PWR014" H 9400 9850 50  0001 C CNN
-F 1 "GND" H 9400 9950 50  0000 C CNN
-F 2 "" H 9400 10100 50  0001 C CNN
-F 3 "" H 9400 10100 50  0001 C CNN
-	1    9400 10100
-	1    0    0    -1
-$EndComp
-Wire Wire Line
-	9950 9900 9400 9900
-Wire Wire Line
-	9400 9900 9400 10100
-Wire Wire Line
-	9400 10000 9950 10000
-Connection ~ 9400 10000
-NoConn ~ 9950 10100
-NoConn ~ 9950 10200
-Text Label 10700 10200 0    60   ~ 0
+P 9400 9800
+F 0 "#PWR014" H 9400 9550 50  0001 C CNN
+F 1 "GND" H 9400 9650 50  0000 C CNN
+F 2 "" H 9400 9800 50  0001 C CNN
+F 3 "" H 9400 9800 50  0001 C CNN
+	1    9400 9800
+	1    0    0    -1
+$EndComp
+Wire Wire Line
+	9950 9600 9400 9600
+Wire Wire Line
+	9400 9600 9400 9800
+Wire Wire Line
+	9400 9700 9950 9700
+Connection ~ 9400 9700
+NoConn ~ 9950 9800
+NoConn ~ 9950 9900
+Text Label 10700 9900 0    60   ~ 0
 STM_NRST
 Wire Wire Line
-	10450 10200 10700 10200
-NoConn ~ 10450 10100
-Text Label 11150 10000 0    60   ~ 0
+	10450 9900 10700 9900
+Text Label 11150 9700 0    60   ~ 0
 TDO
-Text Label 11150 9900 0    60   ~ 0
+Text Label 11150 9600 0    60   ~ 0
 TCK
-Text Label 11150 9800 0    60   ~ 0
+Text Label 11150 9500 0    60   ~ 0
 TMS
 Wire Wire Line
-	10450 10000 11150 10000
-Wire Wire Line
-	10450 9900 11150 9900
-Wire Wire Line
-	10450 9800 11150 9800
-$Comp
-L R R11
-U 1 1 59FB3876
-P 10600 9400
-F 0 "R11" V 10680 9400 50  0000 C CNN
-F 1 "100K" V 10600 9400 50  0000 C CNN
-F 2 "" V 10530 9400 50  0001 C CNN
-F 3 "" H 10600 9400 50  0001 C CNN
-	1    10600 9400
-	1    0    0    -1
-$EndComp
-$Comp
-L R R12
-U 1 1 59FB3C1D
-P 10800 9400
-F 0 "R12" V 10880 9400 50  0000 C CNN
-F 1 "100K" V 10800 9400 50  0000 C CNN
-F 2 "" V 10730 9400 50  0001 C CNN
-F 3 "" H 10800 9400 50  0001 C CNN
-	1    10800 9400
-	1    0    0    -1
-$EndComp
-$Comp
-L R R13
-U 1 1 59FB3C99
-P 11000 9400
-F 0 "R13" V 11080 9400 50  0000 C CNN
-F 1 "100K" V 11000 9400 50  0000 C CNN
-F 2 "" V 10930 9400 50  0001 C CNN
-F 3 "" H 11000 9400 50  0001 C CNN
-	1    11000 9400
-	1    0    0    -1
-$EndComp
-Wire Wire Line
-	11000 9550 11000 9800
-Connection ~ 11000 9800
-Wire Wire Line
-	10800 9550 10800 9900
-Connection ~ 10800 9900
-Wire Wire Line
-	10600 9550 10600 10000
-Connection ~ 10600 10000
-$Comp
-L +3.3V #PWR015
-U 1 1 59FB3FA5
-P 10800 9050
-F 0 "#PWR015" H 10800 8900 50  0001 C CNN
-F 1 "+3.3V" H 10800 9190 50  0000 C CNN
-F 2 "" H 10800 9050 50  0001 C CNN
-F 3 "" H 10800 9050 50  0001 C CNN
-	1    10800 9050
-	1    0    0    -1
-$EndComp
-Wire Wire Line
-	10800 9050 10800 9250
-Wire Wire Line
-	10600 9250 10600 9200
-Wire Wire Line
-	10600 9200 10800 9200
-Connection ~ 10800 9200
-Wire Wire Line
-	10800 9100 11000 9100
-Wire Wire Line
-	11000 9100 11000 9250
-Connection ~ 10800 9100
+	10450 9700 11150 9700
+Wire Wire Line
+	10450 9600 11150 9600
+Wire Wire Line
+	10450 9500 11150 9500
 $Comp
 L +3.3V #PWR016
@@
 	15000 7900 15000 8100
 Connection ~ 15000 8000
-Text Notes 10100 9600 0    60   ~ 0
+Text Notes 10100 9300 0    60   ~ 0
 JTAG
 $Comp
@@
 L Conn_02x05_Odd_Even J3
 U 1 1 59FBB251
-P 10150 10000
-F 0 "J3" H 10200 10300 50  0000 C CNN
-F 1 "Conn_02x05_Odd_Even" H 10200 9700 50  0000 C CNN
-F 2 "" H 10150 10000 50  0001 C CNN
-F 3 "" H 10150 10000 50  0001 C CNN
-	1    10150 10000
+P 10150 9700
+F 0 "J3" H 10200 10000 50  0000 C CNN
+F 1 "Conn_02x05_Odd_Even" H 10200 9400 50  0000 C CNN
+F 2 "" H 10150 9700 50  0001 C CNN
+F 3 "" H 10150 9700 50  0001 C CNN
+	1    10150 9700
 	1    0    0    -1
 $EndComp
@@
 Wire Wire Line
 	5350 7350 5500 7350
-NoConn ~ 5350 7150
 NoConn ~ 5350 6950
 NoConn ~ 5350 9650
@@
 	5200 3300 5200 3800
 Connection ~ 5200 3800
+Text Label 5500 7150 0    60   ~ 0
+TDI
+Wire Wire Line
+	5500 7150 5350 7150
+Text Label 11150 9800 0    60   ~ 0
+TDI
+Wire Wire Line
+	11150 9800 10450 9800
 $EndSCHEMATC

Commit message: Adds ability to reset BLE module using our MCU
Connections:
- net labels added: BLE_nRST
- wire segments 325 -> 326
- no-connect marks 17 -> 16
Changed lines of the file:
@@
 L RT9818A-18GV U7
 U 1 1 59F8E819
-P 13200 7950
-F 0 "U7" H 12900 8300 60  0000 L CNN
-F 1 "RT9818A-18GV" H 12900 8200 60  0000 L CNN
-F 2 "" H 13150 7950 60  0001 C CNN
-F 3 "" H 13150 7950 60  0001 C CNN
-	1    13200 7950
+P 12950 7950
+F 0 "U7" H 12650 8300 60  0000 L CNN
+F 1 "RT9818A-18GV" H 12650 8200 60  0000 L CNN
+F 2 "" H 12900 7950 60  0001 C CNN
+F 3 "" H 12900 7950 60  0001 C CNN
+	1    12950 7950
 	1    0    0    -1
 $EndComp
@@
 L R R24
 U 1 1 59FAE964
-P 13850 7600
-F 0 "R24" V 13930 7600 50  0000 C CNN
-F 1 "4.75K" V 13850 7600 50  0000 C CNN
-F 2 "" V 13780 7600 50  0001 C CNN
-F 3 "" H 13850 7600 50  0001 C CNN
-	1    13850 7600
-	1    0    0    -1
-$EndComp
-Wire Wire Line
-	13700 7850 14100 7850
+P 13600 7600
+F 0 "R24" V 13680 7600 50  0000 C CNN
+F 1 "4.75K" V 13600 7600 50  0000 C CNN
+F 2 "" V 13530 7600 50  0001 C CNN
+F 3 "" H 13600 7600 50  0001 C CNN
+	1    13600 7600
+	1    0    0    -1
+$EndComp
+Wire Wire Line
+	13450 7850 14100 7850
 Wire Wire Line
 	14100 7850 14100 7500
@@
 L C_Small C23
 U 1 1 59FAEA06
-P 13900 8050
-F 0 "C23" H 13910 8120 50  0000 L CNN
-F 1 "1uF" H 13910 7970 50  0000 L CNN
-F 2 "" H 13900 8050 50  0001 C CNN
-F 3 "" H 13900 8050 50  0001 C CNN
-	1    13900 8050
+P 13650 8050
+F 0 "C23" H 13660 8120 50  0000 L CNN
+F 1 "1uF" H 13660 7970 50  0000 L CNN
+F 2 "" H 13650 8050 50  0001 C CNN
+F 3 "" H 13650 8050 50  0001 C CNN
+	1    13650 8050
 	1    0    0    -1
 $EndComp
@@
 L GND #PWR05
 U 1 1 59FAEAA7
-P 13900 8250
-F 0 "#PWR05" H 13900 8000 50  0001 C CNN
-F 1 "GND" H 13900 8100 50  0000 C CNN
-F 2 "" H 13900 8250 50  0001 C CNN
-F 3 "" H 13900 8250 50  0001 C CNN
-	1    13900 8250
+P 13650 8250
+F 0 "#PWR05" H 13650 8000 50  0001 C CNN
+F 1 "GND" H 13650 8100 50  0000 C CNN
+F 2 "" H 13650 8250 50  0001 C CNN
+F 3 "" H 13650 8250 50  0001 C CNN
+	1    13650 8250
 	1    0    0    -1
 $EndComp
@@
 L +3.3V #PWR06
 U 1 1 59FAEB7D
-P 13850 7350
-F 0 "#PWR06" H 13850 7200 50  0001 C CNN
-F 1 "+3.3V" H 13850 7490 50  0000 C CNN
-F 2 "" H 13850 7350 50  0001 C CNN
-F 3 "" H 13850 7350 50  0001 C CNN
-	1    13850 7350
-	1    0    0    -1
-$EndComp
-Wire Wire Line
-	13850 7350 13850 7450
-Wire Wire Line
-	13850 7750 13850 7850
-Connection ~ 13850 7850
-Wire Wire Line
-	13900 7950 13900 7850
-Connection ~ 13900 7850
-Wire Wire Line
-	13900 8150 13900 8250
+P 13600 7350
+F 0 "#PWR06" H 13600 7200 50  0001 C CNN
+F 1 "+3.3V" H 13600 7490 50  0000 C CNN
+F 2 "" H 13600 7350 50  0001 C CNN
+F 3 "" H 13600 7350 50  0001 C CNN
+	1    13600 7350
+	1    0    0    -1
+$EndComp
+Wire Wire Line
+	13600 7350 13600 7450
+Wire Wire Line
+	13600 7750 13600 7850
+Connection ~ 13600 7850
+Wire Wire Line
+	13650 7950 13650 7850
+Connection ~ 13650 7850
+Wire Wire Line
+	13650 8150 13650 8250
 $Comp
 L GND #PWR07
 U 1 1 59FAEF16
-P 13200 8500
-F 0 "#PWR07" H 13200 8250 50  0001 C CNN
-F 1 "GND" H 13200 8350 50  0000 C CNN
-F 2 "" H 13200 8500 50  0001 C CNN
-F 3 "" H 13200 8500 50  0001 C CNN
-	1    13200 8500
-	1    0    0    -1
-$EndComp
-Wire Wire Line
-	13200 8500 13200 8350
+P 12950 8500
+F 0 "#PWR07" H 12950 8250 50  0001 C CNN
+F 1 "GND" H 12950 8350 50  0000 C CNN
+F 2 "" H 12950 8500 50  0001 C CNN
+F 3 "" H 12950 8500 50  0001 C CNN
+	1    12950 8500
+	1    0    0    -1
+$EndComp
+Wire Wire Line
+	12950 8500 12950 8350
 $Comp
 L +3.3V #PWR08
 U 1 1 59FAF139
-P 12600 7750
-F 0 "#PWR08" H 12600 7600 50  0001 C CNN
-F 1 "+3.3V" H 12600 7890 50  0000 C CNN
-F 2 "" H 12600 7750 50  0001 C CNN
-F 3 "" H 12600 7750 50  0001 C CNN
-	1    12600 7750
-	1    0    0    -1
-$EndComp
-Wire Wire Line
-	12600 7750 12600 7850
-Wire Wire Line
-	12600 7850 12700 7850
+P 12350 7750
+F 0 "#PWR08" H 12350 7600 50  0001 C CNN
+F 1 "+3.3V" H 12350 7890 50  0000 C CNN
+F 2 "" H 12350 7750 50  0001 C CNN
+F 3 "" H 12350 7750 50  0001 C CNN
+	1    12350 7750
+	1    0    0    -1
+$EndComp
+Wire Wire Line
+	12350 7750 12350 7850
+Wire Wire Line
+	12350 7850 12450 7850
 $Comp
 L +3.3V #PWR09
@@
 Wire Wire Line
 	5350 8450 5600 8450
-Text Label 14150 2200 0    60   ~ 0
+Text Label 14350 2200 2    60   ~ 0
 IMU_SDO
-Text Label 14150 2700 0    60   ~ 0
+Text Label 14350 2700 2    60   ~ 0
 IMU_SDI
-Wire Wire Line
-	14150 2700 14550 2700
-Wire Wire Line
-	14150 2200 14550 2200
-Text Label 14150 2600 0    60   ~ 0
+Text Label 14350 2600 2    60   ~ 0
 IMU_SCL
-Wire Wire Line
-	14150 2600 14550 2600
 $Comp
 L +3.3V #PWR023
@@
 	5350 7350 5500 7350
 NoConn ~ 5350 6950
-NoConn ~ 5350 9650
 $Comp
 L TPS60241DGKR U6
@@
 Text Label 14350 2400 2    60   ~ 0
 IMU_INT_2
-Wire Wire Line
-	14350 2400 14550 2400
-Wire Wire Line
-	14350 2300 14550 2300
 NoConn ~ 5350 9150
 NoConn ~ 5350 8250
@@
 Wire Notes Line
 	5050 600  5050 2500
-Text Label 14150 2500 0    60   ~ 0
+Text Label 14350 2500 2    60   ~ 0
 IMU_CS
-Wire Wire Line
-	14150 2500 14550 2500
 Text Label 14850 4650 0    60   ~ 0
 DISP_SCS
@@
 Wire Wire Line
 	11150 9800 10450 9800
+Text Label 14100 7500 2    60   ~ 0
+BLE_nRST
+Text Label 5600 9650 0    60   ~ 0
+BLE_nRST
+Wire Wire Line
+	5350 9650 5600 9650
+Wire Wire Line
+	14350 2700 14550 2700
+Wire Wire Line
+	14550 2600 14350 2600
+Wire Wire Line
+	14350 2500 14550 2500
+Wire Wire Line
+	14550 2400 14350 2400
+Wire Wire Line
+	14350 2300 14550 2300
+Wire Wire Line
+	14550 2200 14350 2200
 $EndSCHEMATC

Commit message: Associating most of the footprints.
Parts:
- C1, C10, C11, C13, C15, C16, C17, C2, C21, C25, C26, C27, C3, C4, C9: footprint (none) -> Capacitors_SMD:C_0603
- C12, C14, C18, C19, C20, C22, C23, C24, C5, C6, C7, C8: footprint (none) -> Capacitors_SMD:C_0805
- D1, D4: footprint (none) -> LEDs:LED_0805
- FP1: footprint (none) -> open_watch:BM71BLES1FC2
- J1: footprint (none) -> open_watch:USB_microB_2040002-1
- J3: footprint (none) -> Pin_Headers:Pin_Header_Straight_2x05_Pitch1.00mm
- J4: footprint (none) -> Pin_Headers:Pin_Header_Straight_1x02_Pitch1.00mm
- J6: footprint (none) -> Pin_Headers:Pin_Header_Straight_1x05_Pitch1.00mm
- R1, R10, R14, R15, R16, R17, R18, R19, R2, R20, R21, R22, R23, R24, R25, R3, R4, R5, R6, R7, R8, R9: footprint (none) -> Resistors_SMD:R_0603
- U1: footprint (none) -> Housings_QFP:LQFP-48_7x7mm_Pitch0.5mm
- U3: footprint (none) -> TO_SOT_Packages_SMD:SOT-23-5
- U7: footprint (none) -> TO_SOT_Packages_SMD:SOT-23

Commit message: Adds additional footprint associations
Parts:
- BT1: footprint (none) -> open_watch:BH3000
Connections:
- net labels added: BLE_CONF
- no-connect marks 16 -> 15
Changed lines of the file:
@@
 	15400 6350 15400 6250
-$Comp
-L +3.3V #PWR011
-U 1 1 59FAFE76
-P 15900 6750
-F 0 "#PWR011" H 15900 6600 50  0001 C CNN
-F 1 "+3.3V" H 15900 6890 50  0000 C CNN
-F 2 "" H 15900 6750 50  0001 C CNN
-F 3 "" H 15900 6750 50  0001 C CNN
-	1    15900 6750
-	1    0    0    -1
-$EndComp
-Wire Wire Line
-	15600 7000 15900 7000
-Wire Wire Line
-	15900 7000 15900 6750
 $Comp
 L LED D4
@@
 Wire Wire Line
 	5350 7350 5500 7350
-NoConn ~ 5350 6950
 $Comp
 L TPS60241DGKR U6
@@
 F 0 "BT1" H 1800 3700 50  0000 L CNN
 F 1 "Battery_Cell" H 1800 3600 50  0000 L CNN
-F 2 "" V 1700 3660 50  0001 C CNN
+F 2 "open_watch:BH3000" V 1700 3660 50  0001 C CNN
 F 3 "" V 1700 3660 50  0001 C CNN
 	1    1700 3600
@@
 Wire Wire Line
 	14550 2200 14350 2200
+Text Label 15700 7000 0    60   ~ 0
+BLE_CONF
+Wire Wire Line
+	15700 7000 15600 7000
+Text Label 5500 6950 0    60   ~ 0
+BLE_CONF
+Wire Wire Line
+	5350 6950 5500 6950
 $EndSCHEMATC

Commit message: Associates more footprints
Parts:
- removed J2: Conn_01x02, symbol Conn_01x02
- removed J5: Conn_01x03, symbol Conn_01x03
- added R11, R12: DNP-0, Resistors_SMD:R_0603, symbol R
- D2: footprint (none) -> open_watch:SMLP34RGB2W3
- D3: footprint (none) -> TO_SOT_Packages_SMD:SOT-23
- J7: footprint (none) -> Pin_Headers:Pin_Header_Straight_1x02_Pitch1.00mm
- Q1, Q2, Q3: footprint (none) -> open_watch:VMT3
- Y1: footprint (none) -> open_watch:ECX-31B
- Y2: footprint (none) -> Crystals:Crystal_SMD_SeikoEpson_FA238V-4pin_3.2x2.5mm
Connections:
- wire segments 326 -> 325
- no-connect marks 15 -> 14

Commit message: Adds footprint associations
Parts:
- U2: value TPS2112APWR -> TPS2113ADRBR; footprint (none) -> open_watch:SON-8
- U5: footprint (none) -> open_watch:AT42QT1070-MMHR
Changed lines of the file:
@@
 F 0 "U5" H 10450 2050 60  0000 L CNN
 F 1 "AT42QT1070-MMHR" H 10350 1950 60  0000 L CNN
-F 2 "" H 10400 1850 60  0001 C CNN
+F 2 "open_watch:AT42QT1070-MMHR" H 10400 1850 60  0001 C CNN
 F 3 "" H 10400 1850 60  0001 C CNN
 	1    10400 1850
@@
 P 3850 3800
 F 0 "U2" H 4050 4050 60  0000 L CNN
-F 1 "TPS2112APWR" H 4050 3950 60  0000 L CNN
-F 2 "" H 3850 3800 60  0001 C CNN
+F 1 "TPS2113ADRBR " H 4050 3950 60  0000 L CNN
+F 2 "open_watch:SON-8" H 3850 3800 60  0001 C CNN
 F 3 "" H 3850 3800 60  0001 C CNN
 	1    3850 3800

Commit message: Associates more footprints
Parts:
- U4: footprint (none) -> TO_SOT_Packages_SMD:SOT-23-5
- U9: footprint (none) -> Housings_LGA:Bosch_LGA-14_3x2.5mm_Pitch0.5mm

Commit message: Associates all footprints
Parts:
- SW1, SW2: footprint (none) -> open_watch:PTS820_J15M_SMTR_LFS
- U6: footprint (none) -> Housings_SSOP:MSOP-8_3x3mm_Pitch0.65mm
- U8: footprint (none) -> open_watch:Molex_FPC_5034801000
Changed lines of the file:
@@
 F 0 "U8" H 13650 4600 60  0000 L CNN
 F 1 "WM1389CT-ND" H 13650 4500 60  0000 L CNN
-F 2 "" H 13450 4350 60  0001 C CNN
+F 2 "open_watch:Molex_FPC_5034801000" H 13450 4350 60  0001 C CNN
 F 3 "" H 13450 4350 60  0001 C CNN
 	1    13450 4350
@@
 F 0 "SW1" H 1600 7350 50  0000 L CNN
 F 1 "SW_Push" H 1550 7190 50  0000 C CNN
-F 2 "" H 1550 7450 50  0001 C CNN
+F 2 "open_watch:PTS820_J15M_SMTR_LFS" H 1550 7450 50  0001 C CNN
 F 3 "" H 1550 7450 50  0001 C CNN
 	1    1550 7250
@@
 F 0 "U6" H 10600 4650 60  0000 L CNN
 F 1 "TPS60241DGKR" H 10600 4550 60  0000 L CNN
-F 2 "" H 10400 4400 60  0001 C CNN
+F 2 "Housings_SSOP:MSOP-8_3x3mm_Pitch0.65mm" H 10400 4400 60  0001 C CNN
 F 3 "" H 10400 4400 60  0001 C CNN
 	1    10400 4400
@@
 F 0 "SW2" H 2250 7250 50  0000 L CNN
 F 1 "SW_Push" H 2200 7090 50  0000 C CNN
-F 2 "" H 2200 7350 50  0001 C CNN
+F 2 "open_watch:PTS820_J15M_SMTR_LFS" H 2200 7350 50  0001 C CNN
 F 3 "" H 2200 7350 50  0001 C CNN
 	1    2200 7150
