File: kicad/OpenWatch.sch (KiCad schematic (older format))
At the start: 78 parts, among them J1 USB_microB_2040002-1, J3 Conn_02x05_Odd_Even, J4 Vibration Motor, J6 Conn_01x05, J7 Conn_01x02, Q1 RUM002N02T2L, Q2 RUM002N02T2L, Q3 RUM002N02T2L, SW1 SW_Push, SW2 SW_Push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

Commit message: Fix connections to display
Parts:
- removed J7: Conn_01x02, Pin_Headers:Pin_Header_Straight_1x02_Pitch1.00mm, symbol Conn_01x02
Connections:
- net labels added: EXTCOMIN
- wire segments 325 -> 323
- no-connect marks 14 -> 15
Changed lines of the file:
@@
 	5550 8950 5350 8950
 Wire Wire Line
-	5550 8850 5350 8850
-Wire Wire Line
-	5550 9050 5350 9050
+	5350 8850 6000 8850
+Wire Wire Line
+	5350 9050 6000 9050
 $Comp
 L WM1389CT-ND U8
@@
 Text Notes 13500 5200 0    60   ~ 0
 -What is EXTCOMIN used for?\n-How do we verify the pitch for the FPC?\n
-Text Label 5550 7950 0    60   ~ 0
+Text Label 6000 8850 0    60   ~ 0
 DISP_SDI
-Text Label 5550 8150 0    60   ~ 0
+Text Label 6000 9050 0    60   ~ 0
 DISP_SCLK
-Wire Wire Line
-	5350 8150 5550 8150
-Wire Wire Line
-	5550 7950 5350 7950
 $Comp
 L GND #PWR030
@@
 Wire Wire Line
 	2700 6150 2700 6850
-NoConn ~ 5350 8050
 Wire Wire Line
 	5350 7050 5500 7050
@@
 Text Notes 900  5600 0    60   ~ 0
 Microcontroller\n
-$Comp
-L Conn_01x02 J7
-U 1 1 59FEEB4F
-P 15050 4000
-F 0 "J7" V 15050 4100 50  0000 C CNN
-F 1 "Conn_01x02" V 15050 3550 50  0000 C CNN
-F 2 "Pin_Headers:Pin_Header_Straight_1x02_Pitch1.00mm" H 15050 4000 50  0001 C CNN
-F 3 "" H 15050 4000 50  0001 C CNN
-	1    15050 4000
-	0    -1   -1   0
-$EndComp
-Wire Wire Line
-	14650 4350 15050 4350
-Wire Wire Line
-	15050 4350 15050 4200
-Wire Wire Line
-	14650 4550 15150 4550
-Wire Wire Line
-	15150 4550 15150 4200
+Wire Wire Line
+	15050 4350 14650 4350
+Wire Wire Line
+	15050 4100 15050 4350
 $Comp
 L TSP70933DBVR U3
@@
 IMU_INT_2
 NoConn ~ 5350 9150
-NoConn ~ 5350 8250
 $Comp
 L GND #PWR059
@@
 Wire Wire Line
 	12150 4150 12200 4150
+$Comp
+L +5V #PWR?
+U 1 1 5A0A3934
+P 15050 4100
+F 0 "#PWR?" H 15050 3950 50  0001 C CNN
+F 1 "+5V" H 15050 4240 50  0000 C CNN
+F 2 "" H 15050 4100 50  0001 C CNN
+F 3 "" H 15050 4100 50  0001 C CNN
+	1    15050 4100
+	1    0    0    -1
+$EndComp
+Wire Wire Line
+	14650 4550 14850 4550
+Text Label 14850 4550 0    60   ~ 0
+EXTCOMIN
+Text Label 5550 7950 0    60   ~ 0
+EXTCOMIN
+Wire Wire Line
+	5550 7950 5350 7950
+NoConn ~ 5350 8050
+NoConn ~ 5350 8150
+NoConn ~ 5350 8250
 $EndSCHEMATC

Commit message: Fix various connection issues
Parts:
- removed R12: DNP-0, Resistors_SMD:R_0603, symbol R
Connections:
- net labels added: DISP_EN
- wire segments 323 -> 322
- no-connect marks 15 -> 14
Changed lines of the file:
@@
 L +5V #PWR044
 U 1 1 59FE5F7E
-P 12150 4000
-F 0 "#PWR044" H 12150 3850 50  0001 C CNN
-F 1 "+5V" H 12150 4140 50  0000 C CNN
-F 2 "" H 12150 4000 50  0001 C CNN
-F 3 "" H 12150 4000 50  0001 C CNN
-	1    12150 4000
+P 12500 4150
+F 0 "#PWR044" H 12500 4000 50  0001 C CNN
+F 1 "+5V" H 12500 4290 50  0000 C CNN
+F 2 "" H 12500 4150 50  0001 C CNN
+F 3 "" H 12500 4150 50  0001 C CNN
+	1    12500 4150
 	1    0    0    -1
 $EndComp
@@
 	8600 3900 8600 3750
 $Comp
-L R R12
-U 1 1 5A07BCA5
-P 12350 4150
-F 0 "R12" V 12430 4150 50  0000 C CNN
-F 1 "DNP-0" V 12350 4150 50  0000 C CNN
-F 2 "Resistors_SMD:R_0603" V 12280 4150 50  0001 C CNN
-F 3 "" H 12350 4150 50  0001 C CNN
-	1    12350 4150
-	0    1    1    0
-$EndComp
-Wire Wire Line
-	12150 4000 12150 4150
-Wire Wire Line
-	12150 4150 12200 4150
-$Comp
-L +5V #PWR?
+L +5V #PWR061
 U 1 1 5A0A3934
 P 15050 4100
-F 0 "#PWR?" H 15050 3950 50  0001 C CNN
+F 0 "#PWR061" H 15050 3950 50  0001 C CNN
 F 1 "+5V" H 15050 4240 50  0000 C CNN
 F 2 "" H 15050 4100 50  0001 C CNN
@@
 Wire Wire Line
 	5550 7950 5350 7950
-NoConn ~ 5350 8050
 NoConn ~ 5350 8150
 NoConn ~ 5350 8250
+Text Label 15650 4450 0    60   ~ 0
+DISP_EN
+Text Label 5550 8050 0    60   ~ 0
+DISP_EN
+Wire Wire Line
+	5350 8050 5550 8050
 $EndSCHEMATC

Commit message: Fix no pull down on transistor gates
Parts:
- added R12, R13, R26: 100K, Resistors_SMD:R_0603, symbol R
- BT1: footprint open_watch:BH3000 -> open_watch:Molex-0532610271
Connections:
- wire segments 322 -> 330

Commit message: Change battery connector to two holes
Parts:
- BT1: footprint open_watch:Molex-0532610271 -> Pin_Headers:Pin_Header_Straight_1x02_Pitch2.00mm
Connections:
- net labels added: D_N, D_P
- net labels removed: D+, D-
Changed lines of the file:
@@
 Connection ~ 1800 1850
 Text Label 2825 1100 0    60   ~ 0
-D+
+D_N
 Text Label 2825 1200 0    60   ~ 0
-D-
+D_P
 Wire Wire Line
 	2825 1200 2700 1200
@@
 F 0 "BT1" H 1800 3700 50  0000 L CNN
 F 1 "Battery_Cell" H 1800 3600 50  0000 L CNN
-F 2 "open_watch:Molex-0532610271" V 1700 3660 50  0001 C CNN
+F 2 "Pin_Headers:Pin_Header_Straight_1x02_Pitch2.00mm" V 1700 3660 50  0001 C CNN
 F 3 "" V 1700 3660 50  0001 C CNN
 	1    1700 3600
@@
 Bypass Capacitors\n
 Text Label 5500 7550 0    60   ~ 0
-D-
+D_N
 Wire Wire Line
 	5350 7550 5500 7550
 Text Label 5500 7450 0    60   ~ 0
-D+
+D_P
 Wire Wire Line
 	5500 7450 5350 7450

Commit message: Finish majority of routing
Changed lines of the file:
@@
 Text Label 2300 4100 0    60   ~ 0
 BATT_EN
-Text Label 5600 9350 0    60   ~ 0
+Text Label 5500 6950 0    60   ~ 0
 BATT_EN
-Wire Wire Line
-	5350 9350 5600 9350
 Text Notes 1500 5150 0    60   ~ 0
 Allow for\ncompletely\nturning off \nthe battery\n
@@
 Wire Wire Line
 	5600 8150 5350 8150
-NoConn ~ 5350 6950
+Wire Wire Line
+	5500 6950 5350 6950
+NoConn ~ 5350 9350
 $EndSCHEMATC
